File: hardware/AcousticSpeedCameraShield/mcu_conn.kicad_sch (KiCad schematic)
At the start: 2 parts, among them CN11 Conn_02x36_Odd_Even, CN12 Conn_02x36_Odd_Even

Commit message: update MCU pin assignments
Connections:
- net CAM_HSYNC: now reaches CN11.32 (Pin_32)
- net VBAT_RTC: now reaches CN11.33 (Pin_33)
- net ADC3_INP10: now reaches CN11.38 (Pin_38)
- net DISP_CS: now reaches CN11.4 (Pin_4)
- net CAM_D5: now reaches CN11.40 (Pin_40)
- net PDM_DAT4: now reaches CN11.45 (Pin_45)
- net CAM_D4: now reaches CN11.48 (Pin_48)
- net CAM_D6: now reaches CN11.50 (Pin_50)
- net DISP_RST: now reaches CN11.61 (Pin_61)
- net CAM_VSYNC: now reaches CN11.63 (Pin_63)
- net CAM_PIXCLK: now reaches CN12.13 (Pin_13)
- net CAM_XCLK: now reaches CN12.23 (Pin_23)
- net CAM_D2: now reaches CN12.30 (Pin_30)
- net CAM_D7: now reaches CN12.5 (Pin_5)
- net CAM_PWDN: now reaches CN12.68 (Pin_68)
- net CAM_RST: now reaches CN12.69 (Pin_69)
- net LCD_BL renamed DISP_BL
- net LCD_CLK renamed DISP_CLK
- net LCD_CS renamed CAM_D0
- net LCD_DC renamed DISP_DC
- net LCD_DIN renamed DISP_DIN
- net LCD_RST renamed CAM_D3
- net PDM_DAT2 renamed CAM_D1
- no-connect marks 113 -> 97
Other:
- title: (none) -> Złącza Mikrokontrolera
